Commit message: Works with ARMSTONE!

File: urdf/armstone/as.urdf (robot description, URDF)
Before this commit: robot armstone, 25 links, 24 joints
Links:
- link xarmlink1: geometry collision mesh filename=package://perceptive_mpc/urdf/armstone/meshes/xarm6/visual/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; visual mesh filename=package://perceptive_mpc/urdf/armstone/meshes/xarm6/visual/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
- link xarmlink2: geometry collision mesh filename=package://perceptive_mpc/urdf/armstone/meshes/xarm6/visual/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; visual mesh filename=package://perceptive_mpc/urdf/armstone/meshes/xarm6/visual/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
- link xarmlink3: geometry collision mesh filename=package://perceptive_mpc/urdf/armstone/meshes/xarm6/visual/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; visual mesh filename=package://perceptive_mpc/urdf/armstone/meshes/xarm6/visual/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
- link xarmlink4: geometry collision mesh filename=package://perceptive_mpc/urdf/armstone/meshes/xarm6/visual/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; visual mesh filename=package://perceptive_mpc/urdf/armstone/meshes/xarm6/visual/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
- link xarmlink5: geometry collision mesh filename=package://perceptive_mpc/urdf/armstone/meshes/xarm6/visual/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; visual mesh filename=package://perceptive_mpc/urdf/armstone/meshes/xarm6/visual/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
- link xarmlink6: geometry collision mesh filename=package://perceptive_mpc/urdf/armstone/meshes/xarm6/visual/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; visual mesh filename=package://perceptive_mpc/urdf/armstone/meshes/xarm6/visual/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
- link xarmlink_base: geometry collision mesh filename=package://perceptive_mpc/urdf/armstone/meshes/xarm6/visual/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; visual mesh filename=package://perceptive_mpc/urdf/armstone/meshes/xarm6/visual/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
